File: hardware/gswitch18.kicad_sch (KiCad schematic)
At the start: 25 parts, among them IC1 ATMEGA88P, P1 CONN_6X2, P2 CONN_6X2, P3 CONN_6X2, P4 USB, P5 ISP, X1 12MHz

Commit message: v1.2 final tidy-up
Other:
- title: G9X USB Programmer -> https://github.com/gruvin/gswitch18
